File: board/plc14500/SPRAM.kicad_sch (KiCad schematic)
At the start: 30 parts, among them U12 4011, U13 4099, U14 4051

Commit message: Fixes
Changed lines of the file:
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@@
     (comment 1 "REV.D")
   )
-  (junction (at 199.39 149.86) (diameter 0) (color 0 0 0 0)
-  )
   (junction (at 214.63 92.71) (diameter 0) (color 0 0 0 0)
   )
-  (junction (at 190.5 149.86) (diameter 0) (color 0 0 0 0)
+  (junction (at 190.5 151.13) (diameter 0) (color 0 0 0 0)
   )
   (junction (at 229.87 62.23) (diameter 0) (color 0 0 0 0)
   )
-  (junction (at 190.5 124.46) (diameter 0) (color 0 0 0 0)
+  (junction (at 190.5 122.555) (diameter 0) (color 0 0 0 0)
   )
   (junction (at 224.79 59.69) (diameter 0) (color 0 0 0 0)
@@
   (junction (at 182.88 36.83) (diameter 0) (color 0 0 0 0)
   )
+  (junction (at 199.39 151.13) (diameter 0) (color 0 0 0 0)
+  )
   (junction (at 224.79 92.71) (diameter 0) (color 0 0 0 0)
   )
@@
   (junction (at 209.55 52.07) (diameter 0) (color 0 0 0 0)
   )
-  (junction (at 194.31 149.86) (diameter 0) (color 0 0 0 0)
+  (junction (at 194.31 151.13) (diameter 0) (color 0 0 0 0)
   )
   (junction (at 204.47 49.53) (diameter 0) (color 0 0 0 0)
   )
-  (junction (at 194.31 124.46) (diameter 0) (color 0 0 0 0)
+  (junction (at 194.31 122.555) (diameter 0) (color 0 0 0 0)
   )
   (junction (at 100.965 95.25) (diameter 0) (color 0 0 0 0)
@@
   (junction (at 219.71 92.71) (diameter 0) (color 0 0 0 0)
   )
-  (junction (at 199.39 124.46) (diameter 0) (color 0 0 0 0)
+  (junction (at 199.39 122.555) (diameter 0) (color 0 0 0 0)
   )
   (junction (at 102.235 127) (diameter 0) (color 0 0 0 0)
@@
     (stroke (width 0) (type default))
   )
-  (wire (pts (xy 199.39 124.46) (xy 205.74 124.46))
+  (wire (pts (xy 194.31 122.555) (xy 199.39 122.555))
     (stroke (width 0) (type default))
   )
@@
     (stroke (width 0) (type default))
   )
-  (wire (pts (xy 194.31 149.86) (xy 199.39 149.86))
+  (wire (pts (xy 194.31 151.13) (xy 199.39 151.13))
     (stroke (width 0) (type default))
   )
@@
     (stroke (width 0) (type default))
   )
-  (wire (pts (xy 190.5 124.46) (xy 190.5 134.62))
+  (wire (pts (xy 190.5 122.555) (xy 190.5 134.62))
     (stroke (width 0) (type default))
   )
@@
     (stroke (width 0) (type default))
   )
-  (wire (pts (xy 182.88 124.46) (xy 190.5 124.46))
+  (wire (pts (xy 182.88 122.555) (xy 190.5 122.555))
     (stroke (width 0) (type default))
   )
@@
     (stroke (width 0) (type default))
   )
+  (wire (pts (xy 182.88 122.555) (xy 182.88 124.46))
+    (stroke (width 0) (type default))
+  )
   (wire (pts (xy 260.35 85.09) (xy 261.62 85.09))
     (stroke (width 0) (type default))
@@
     (stroke (width 0) (type default))
   )
-  (wire (pts (xy 194.31 149.86) (xy 194.31 153.67))
+  (wire (pts (xy 194.31 151.13) (xy 194.31 153.67))
     (stroke (width 0) (type default))
   )
@@
     (stroke (width 0) (type default))
   )
+  (wire (pts (xy 199.39 122.555) (xy 199.39 124.46))
+    (stroke (width 0) (type default))
+  )
   (wire (pts (xy 74.295 127) (xy 85.725 127))
     (stroke (width 0) (type default))
@@
     (stroke (width 0) (type default))
   )
-  (wire (pts (xy 194.31 124.46) (xy 199.39 124.46))
-    (stroke (width 0) (type default))
-  )
   (wire (pts (xy 100.965 100.33) (xy 104.775 100.33))
     (stroke (width 0) (type default))
@@
     (stroke (width 0) (type default))
   )
-  (wire (pts (xy 205.74 142.24) (xy 205.74 149.86))
-    (stroke (width 0) (type default))
-  )
   (wire (pts (xy 261.62 85.09) (xy 262.89 85.09))
     (stroke (width 0) (type default))
@@
     (stroke (width 0) (type default))
   )
-  (wire (pts (xy 194.31 119.38) (xy 194.31 124.46))
+  (wire (pts (xy 194.31 117.475) (xy 194.31 122.555))
     (stroke (width 0) (type default))
   )
@@
     (stroke (width 0) (type default))
   )
-  (wire (pts (xy 205.74 124.46) (xy 205.74 134.62))
+  (wire (pts (xy 205.74 122.555) (xy 205.74 134.62))
     (stroke (width 0) (type default))
   )
@@
     (stroke (width 0) (type default))
   )
+  (wire (pts (xy 199.39 151.13) (xy 205.74 151.13))
+    (stroke (width 0) (type default))
+  )
   (wire (pts (xy 229.87 62.23) (xy 247.65 62.23))
     (stroke (width 0) (type default))
@@
     (stroke (width 0) (type default))
   )
-  (wire (pts (xy 190.5 142.24) (xy 190.5 149.86))
-    (stroke (width 0) (type default))
-  )
   (wire (pts (xy 160.02 58.42) (xy 172.72 58.42))
     (stroke (width 0) (type default))
@@
     (stroke (width 0) (type default))
   )
-  (wire (pts (xy 182.88 149.86) (xy 190.5 149.86))
+  (wire (pts (xy 199.39 149.86) (xy 199.39 151.13))
+    (stroke (width 0) (type default))
+  )
+  (wire (pts (xy 182.88 151.13) (xy 190.5 151.13))
     (stroke (width 0) (type default))
   )
@@
     (stroke (width 0) (type default))
   )
+  (wire (pts (xy 190.5 142.24) (xy 190.5 151.13))
+    (stroke (width 0) (type default))
+  )
   (wire (pts (xy 191.77 46.99) (xy 199.39 46.99))
     (stroke (width 0) (type default))
@@
     (stroke (width 0) (type default))
   )
-  (wire (pts (xy 190.5 124.46) (xy 194.31 124.46))
+  (wire (pts (xy 190.5 122.555) (xy 194.31 122.555))
     (stroke (width 0) (type default))
   )
@@
     (stroke (width 0) (type default))
   )
-  (wire (pts (xy 199.39 149.86) (xy 205.74 149.86))
-    (stroke (width 0) (type default))
-  )
   (wire (pts (xy 104.775 90.17) (xy 100.965 90.17))
     (stroke (width 0) (type default))
@@
     (stroke (width 0) (type default))
   )
+  (wire (pts (xy 182.88 151.13) (xy 182.88 149.86))
+    (stroke (width 0) (type default))
+  )
   (wire (pts (xy 224.79 88.9) (xy 224.79 92.71))
     (stroke (width 0) (type default))
@@
     (stroke (width 0) (type default))
   )
+  (wire (pts (xy 199.39 122.555) (xy 205.74 122.555))
+    (stroke (width 0) (type default))
+  )
   (wire (pts (xy 104.775 121.92) (xy 102.235 121.92))
     (stroke (width 0) (type default))
@@
     (stroke (width 0) (type default))
   )
+  (wire (pts (xy 205.74 142.24) (xy 205.74 151.13))
+    (stroke (width 0) (type default))
+  )
   (wire (pts (xy 191.77 62.23) (xy 229.87 62.23))
     (stroke (width 0) (type default))
@@
     (stroke (width 0) (type default))
   )
-  (wire (pts (xy 190.5 149.86) (xy 194.31 149.86))
+  (wire (pts (xy 190.5 151.13) (xy 194.31 151.13))
     (stroke (width 0) (type default))
   )
@@
     )
   )
-  (symbol (lib_id "power:+5V") (at 194.31 119.38 0) (unit 1)
-    (in_bom yes) (on_board yes) (dnp no)
-    (property "Reference" "#PWR?" (at 194.31 123.19 0)
-      (effects (font (size 1.27 1.27)) hide)
-    )
-    (property "Value" "+5V" (at 192.405 116.205 90)
-      (effects (font (size 1.27 1.27)))
-    )
-    (property "Footprint" "" (at 194.31 119.38 0)
-      (effects (font (size 1.27 1.27)) hide)
-    )
-    (property "Datasheet" "" (at 194.31 119.38 0)
-      (effects (font (size 1.27 1.27)) hide)
-    )
+  (symbol (lib_id "power:+5V") (at 194.31 117.475 0) (unit 1)
+    (in_bom yes) (on_board yes) (dnp no)
+    (property "Reference" "#PWR?" (at 194.31 121.285 0)
+      (effects (font (size 1.27 1.27)) hide)
+    )
+    (property "Value" "+5V" (at 192.405 114.3 90)
+      (effects (font (size 1.27 1.27)))
+    )
+    (property "Footprint" "" (at 194.31 117.475 0)
+      (effects (font (size 1.27 1.27)) hide)
+    )
+    (property "Datasheet" "" (at 194.31 117.475 0)
+      (effects (font (size 1.27 1.27)) hide)
+    )
