File: board/plc14500/IO.kicad_sch (KiCad schematic)
At the start: 72 parts, among them U1 74HC14, U2 4051, U3 74HC14, U5 4099

Commit message: Cleanup, ready to route
Parts:
- D1, D10, D11, D12, D13, D14, D15, D16, D2, D3, D4, D5, D6, D7, D8, D9: footprint LED_5MM -> plc14500:LED_3MM; Field4 XXX-00000 -> (none)
- J1: footprint (none) -> plc14500:PLC14500-Expansion
Changed lines of the file:
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@@
       (effects (font (size 1.143 1.143)) (justify left) hide)
     )
-    (property "Footprint" "LED_5MM" (at 215.9 63.5 90)
+    (property "Footprint" "plc14500:LED_3MM" (at 215.9 63.5 90)
       (effects (font (size 0.508 0.508)) hide)
     )
@@
       (effects (font (size 1.27 1.27)) hide)
     )
-    (property "Field4" "XXX-00000" (at 214.63 63.5 90)
+    (property "Field4" "" (at 214.63 63.5 90)
       (effects (font (size 1.524 1.524)) hide)
     )
@@
       (effects (font (size 1.143 1.143)) (justify left) hide)
     )
-    (property "Footprint" "LED_5MM" (at 57.15 43.18 90)
+    (property "Footprint" "plc14500:LED_3MM" (at 57.15 43.18 90)
       (effects (font (size 0.508 0.508)) hide)
     )
@@
       (effects (font (size 1.27 1.27)) hide)
     )
-    (property "Field4" "XXX-00000" (at 57.15 41.91 90)
+    (property "Field4" "" (at 57.15 41.91 90)
       (effects (font (size 1.524 1.524)) hide)
     )
@@
       (effects (font (size 1.143 1.143)) (justify left) hide)
     )
-    (property "Footprint" "LED_5MM" (at 180.34 63.5 90)
+    (property "Footprint" "plc14500:LED_3MM" (at 180.34 63.5 90)
       (effects (font (size 0.508 0.508)) hide)
     )
@@
       (effects (font (size 1.27 1.27)) hide)
     )
-    (property "Field4" "XXX-00000" (at 179.07 63.5 90)
+    (property "Field4" "" (at 179.07 63.5 90)
       (effects (font (size 1.524 1.524)) hide)
     )
@@
       (effects (font (size 1.143 1.143)) (justify left) hide)
     )
-    (property "Footprint" "LED_5MM" (at 185.42 63.5 90)
+    (property "Footprint" "plc14500:LED_3MM" (at 185.42 63.5 90)
       (effects (font (size 0.508 0.508)) hide)
     )
@@
       (effects (font (size 1.27 1.27)) hide)
     )
-    (property "Field4" "XXX-00000" (at 184.15 63.5 90)
+    (property "Field4" "" (at 184.15 63.5 90)
       (effects (font (size 1.524 1.524)) hide)
     )
@@
       (effects (font (size 1.143 1.143)) (justify left) hide)
     )
-    (property "Footprint" "LED_5MM" (at 190.5 63.5 90)
+    (property "Footprint" "plc14500:LED_3MM" (at 190.5 63.5 90)
       (effects (font (size 0.508 0.508)) hide)
     )
@@
       (effects (font (size 1.27 1.27)) hide)
     )
-    (property "Field4" "XXX-00000" (at 189.23 63.5 90)
+    (property "Field4" "" (at 189.23 63.5 90)
       (effects (font (size 1.524 1.524)) hide)
     )
@@
       (effects (font (size 1.143 1.143)) (justify left) hide)
     )
-    (property "Footprint" "LED_5MM" (at 195.58 63.5 90)
+    (property "Footprint" "plc14500:LED_3MM" (at 195.58 63.5 90)
       (effects (font (size 0.508 0.508)) hide)
     )
@@
       (effects (font (size 1.27 1.27)) hide)
     )
-    (property "Field4" "XXX-00000" (at 194.31 63.5 90)
+    (property "Field4" "" (at 194.31 63.5 90)
       (effects (font (size 1.524 1.524)) hide)
     )
@@
       (effects (font (size 1.143 1.143)) (justify left) hide)
     )
-    (property "Footprint" "LED_5MM" (at 200.66 63.5 90)
+    (property "Footprint" "plc14500:LED_3MM" (at 200.66 63.5 90)
       (effects (font (size 0.508 0.508)) hide)
     )
@@
       (effects (font (size 1.27 1.27)) hide)
     )
-    (property "Field4" "XXX-00000" (at 199.39 63.5 90)
+    (property "Field4" "" (at 199.39 63.5 90)
       (effects (font (size 1.524 1.524)) hide)
     )
@@
       (effects (font (size 1.143 1.143)) (justify left) hide)
     )
-    (property "Footprint" "LED_5MM" (at 205.74 63.5 90)
+    (property "Footprint" "plc14500:LED_3MM" (at 205.74 63.5 90)
       (effects (font (size 0.508 0.508)) hide)
     )
@@
       (effects (font (size 1.27 1.27)) hide)
     )
-    (property "Field4" "XXX-00000" (at 204.47 63.5 90)
+    (property "Field4" "" (at 204.47 63.5 90)
       (effects (font (size 1.524 1.524)) hide)
     )
@@
       (effects (font (size 1.143 1.143)) (justify left) hide)
     )
-    (property "Footprint" "LED_5MM" (at 210.82 63.5 90)
+    (property "Footprint" "plc14500:LED_3MM" (at 210.82 63.5 90)
       (effects (font (size 0.508 0.508)) hide)
     )
@@
       (effects (font (size 1.27 1.27)) hide)
     )
-    (property "Field4" "XXX-00000" (at 209.55 63.5 90)
+    (property "Field4" "" (at 209.55 63.5 90)
       (effects (font (size 1.524 1.524)) hide)
     )
@@
       (effects (font (size 1.143 1.143)) (justify left) hide)
     )
-    (property "Footprint" "LED_5MM" (at 195.58 134.62 90)
+    (property "Footprint" "plc14500:LED_3MM" (at 195.58 134.62 90)
       (effects (font (size 0.508 0.508)) hide)
     )
@@
       (effects (font (size 1.27 1.27)) hide)
     )
-    (property "Field4" "XXX-00000" (at 194.31 134.62 90)
+    (property "Field4" "" (at 194.31 134.62 90)
       (effects (font (size 1.524 1.524)) hide)
     )
@@
       (effects (font (size 1.143 1.143)) (justify left) hide)
     )
-    (property "Footprint" "LED_5MM" (at 57.15 83.82 90)
+    (property "Footprint" "plc14500:LED_3MM" (at 57.15 83.82 90)
       (effects (font (size 0.508 0.508)) hide)
     )
@@
       (effects (font (size 1.27 1.27)) hide)
     )
-    (property "Field4" "XXX-00000" (at 57.15 82.55 90)
+    (property "Field4" "" (at 57.15 82.55 90)
       (effects (font (size 1.524 1.524)) hide)
     )
@@
       (effects (font (size 1.143 1.143)) (justify left) hide)
     )
-    (property "Footprint" "LED_5MM" (at 57.15 121.92 90)
+    (property "Footprint" "plc14500:LED_3MM" (at 57.15 121.92 90)
       (effects (font (size 0.508 0.508)) hide)
     )
@@
       (effects (font (size 1.27 1.27)) hide)
     )
-    (property "Field4" "XXX-00000" (at 57.15 120.65 90)
+    (property "Field4" "" (at 57.15 120.65 90)
       (effects (font (size 1.524 1.524)) hide)
     )
@@
       (effects (font (size 1.143 1.143)) (justify left) hide)
     )
-    (property "Footprint" "LED_5MM" (at 57.15 158.75 90)
+    (property "Footprint" "plc14500:LED_3MM" (at 57.15 158.75 90)
       (effects (font (size 0.508 0.508)) hide)
     )
@@
       (effects (font (size 1.27 1.27)) hide)
     )
-    (property "Field4" "XXX-00000" (at 57.15 157.48 90)
+    (property "Field4" "" (at 57.15 157.48 90)
       (effects (font (size 1.524 1.524)) hide)
     )
@@
       (effects (font (size 1.143 1.143)) (justify left) hide)
     )
-    (property "Footprint" "LED_5MM" (at 121.92 46.99 90)
+    (property "Footprint" "plc14500:LED_3MM" (at 121.92 46.99 90)
       (effects (font (size 0.508 0.508)) hide)
     )
@@
       (effects (font (size 1.27 1.27)) hide)
     )
-    (property "Field4" "XXX-00000" (at 121.92 45.72 90)
+    (property "Field4" "" (at 121.92 45.72 90)
       (effects (font (size 1.524 1.524)) hide)
     )
@@
       (effects (font (size 1.143 1.143)) (justify left) hide)
     )
-    (property "Footprint" "LED_5MM" (at 121.92 83.82 90)
+    (property "Footprint" "plc14500:LED_3MM" (at 121.92 83.82 90)
       (effects (font (size 0.508 0.508)) hide)
     )
@@
       (effects (font (size 1.27 1.27)) hide)
     )
-    (property "Field4" "XXX-00000" (at 121.92 82.55 90)
+    (property "Field4" "" (at 121.92 82.55 90)
       (effects (font (size 1.524 1.524)) hide)
     )
@@
       (effects (font (size 1.143 1.143)) (justify left) hide)
     )
-    (property "Footprint" "LED_5MM" (at 121.92 121.92 90)
+    (property "Footprint" "plc14500:LED_3MM" (at 121.92 121.92 90)
       (effects (font (size 0.508 0.508)) hide)
     )
@@
       (effects (font (size 1.27 1.27)) hide)
     )
-    (property "Field4" "XXX-00000" (at 121.92 120.65 90)
+    (property "Field4" "" (at 121.92 120.65 90)
       (effects (font (size 1.524 1.524)) hide)
     )
@@
       (effects (font (size 1.27 1.27)))
     )
-    (property "Footprint" "" (at 260.35 91.44 0)
-      (effects (font (size 1.27 1.27)) hide)
-    )
+    (property "Footprint" "plc14500:PLC14500-Expansion" (at 260.35 91.44 0)
+      (effects (font (size 1.27 1.27)) hide)
+    )

Commit message: REV.D first proto
Parts:
- C4: footprint Capacitor_THT:CP_Radial_D8.0mm_P5.00mm -> Capacitor_THT:CP_Radial_D5.0mm_P2.50mm
Connections:
- net GND: now also S12.8 (GND), S12.9 (GND), S13.8 (GND), S13.9 (GND), S14.8 (GND), S14.9 (GND), S5.8 (GND), S5.9 (GND), S6.8 (GND), S6.9 (GND), S7.8 (GND), S7.9 (GND), S8.8 (GND), S8.9 (GND)
Other:
- moved on the sheet: R1, R10, R11, R2, R3, R4, R9, S10, S11, S9
