File: board/plc14500/plc14500.kicad_pcb (KiCad board)
At the start: 2 copper layers, 160.1 x 99.9 mm, 170 parts, among them U1 74HC14, U10 MC14500, U11 74HC14, U12 4011, U13 4099, U14 4051, U2 4051, U3 74HC14, U4 NE555, U5 4099, U6 Arduino Nano, U7 74HC590A, U8 LH5168, U9 NE555

Commit message: Cleanup, ready to route
Parts:
- added J1: ~, plc14500:PLC14500-Expansion, F.Cu at (218.4, 59.7)
- C4: footprint Capacitor_THT:CP_Radial_D5.0mm_P2.50mm -> Capacitor_THT:CP_Radial_D8.0mm_P5.00mm
- moved D19 5.23 mm to (139.1, 58.2)
- moved R29 5.23 mm to (140.3, 61.6)
- moved D33 5.19 mm to (149.2, 58.0)
- moved R45 5.19 mm to (150.5, 61.3)
- moved D18 4.92 mm to (144.1, 58.0)
- moved R28 4.92 mm to (145.4, 61.3)
- moved D28 4.84 mm to (154.2, 58.0)
- moved R40 4.84 mm to (155.5, 61.3)
- moved D38 0.26 mm to (134.2, 58.2)
- moved R52 0.25 mm to (135.4, 61.6)
Connections:
- net !RES renamed /!RES
- net /Input/Output/IN0 renamed /Input-Output/IN0
- net /Input/Output/IN1 renamed /Input-Output/IN1
- net /Input/Output/IN2 renamed /Input-Output/IN2
- net /Input/Output/IN3 renamed /Input-Output/IN3
- net /Input/Output/IN4 renamed /Input-Output/IN4
- net /Input/Output/IN5 renamed /Input-Output/IN5
- net /Input/Output/IN6 renamed /Input-Output/IN6
- net A0 renamed /A0
- net A3 renamed /A3
- net A4 renamed /A4
- net A5 renamed /A5
- net A6 renamed /A6
- net A7 renamed /A7
- net D renamed /D
- net D0 renamed /D0
- net D1 renamed /D1
- net D2 renamed /D2
- net D3 renamed /D3
- net D4 renamed /D4
- net D5 renamed /D5
- net D6 renamed /D6
- net IN-WINH renamed /IN-INH
- net IN7 renamed /Input-Output/IN7
- net JMP renamed /CPU/JMP
- net Net-(R1-Pad2) renamed /Input-Output/EXTIN0
- net Net-(R10-Pad2) renamed /Input-Output/EXTIN5
- net Net-(R11-Pad2) renamed /Input-Output/EXTIN6
- net Net-(R2-Pad2) renamed /Input-Output/EXTIN1
- net Net-(R3-Pad2) renamed /Input-Output/EXTIN2
- net Net-(R4-Pad2) renamed /Input-Output/EXTIN3
- net Net-(R9-Pad2) renamed /Input-Output/EXTIN4
- net Net-(U5-Q0) renamed /Input-Output/OUT0
- net Net-(U5-Q1) renamed /Input-Output/OUT1
- net Net-(U5-Q2) renamed /Input-Output/OUT2
- net Net-(U5-Q3) renamed /Input-Output/OUT3
- net Net-(U5-Q4) renamed /Input-Output/OUT4
- net Net-(U5-Q5) renamed /Input-Output/OUT5
- net Net-(U5-Q6) renamed /Input-Output/OUT6
- net OUT-WD renamed /OUT-WD
- net PRG renamed /PRG
- net RR renamed /RR
- net SPRAM-WINH renamed /SPRAM/SPRAM-INH
- net SRAM-WD renamed /SPRAM/SPRAM-WD
- net TMR0-TRG renamed /TMR0-TRG
- net W renamed /W
- net WEN renamed /!WEN
- C3 pad 1: GND -> +5V
- C3 pad 2: +5V -> GND
- D17 pad A: RES -> /RES
- D22 pad A: A1 -> /A2
- D24 pad A: A2 -> /A1
- D37 pad A: D7 -> /CPU/D7
- D51 pad 2: RES -> /RES
- R26 pad 1: RES -> /RES
- R31 pad 1: Net-(U9-DIS) -> Net-(U9-TRE)
- R31 pad 2: Net-(U9-TRE) -> Net-(U9-DIS)
- S12 pad 5: Net-(S12-Pad5) -> Net-(S12-Pad1)
- S12 pad 7: Net-(S12-Pad3) -> Net-(S12-Pad7)
- S13 pad 5: Net-(S13-Pad5) -> Net-(S13-Pad1)
- S13 pad 7: Net-(S13-Pad3) -> Net-(S13-Pad7)
- S14 pad 5: Net-(S14-Pad5) -> Net-(S14-Pad1)
- S14 pad 7: Net-(S14-Pad3) -> Net-(S14-Pad7)
- S15 pad 1: RES -> /RES
- S16 pad 1: Net-(R28-Pad1) -> Net-(R29-Pad1)
- S16 pad 3: Net-(R29-Pad1) -> Net-(R28-Pad1)
- S16 pad 5: Net-(U9-TRE) -> unconnected-(S16-Pad5)
- S16 pad 7: unconnected-(S16-Pad7) -> Net-(U9-TRE)
- S18 pad 1: Net-(S18-Pad1) -> Net-(U9-OUT)
- S18 pad 3: Net-(U9-OUT) -> Net-(S18-Pad3)
- S18 pad 5: Net-(D33-PadA) -> Net-(D28-PadA)
- S18 pad 7: Net-(D28-PadA) -> Net-(D33-PadA)
- S5 pad 5: Net-(S5-Pad5) -> Net-(S5-Pad1)
- S5 pad 7: Net-(S5-Pad3) -> Net-(S5-Pad1)
- S6 pad 5: Net-(S6-Pad5) -> Net-(S6-Pad1)
- S6 pad 7: Net-(S6-Pad3) -> Net-(S6-Pad1)
- S7 pad 5: Net-(S7-Pad5) -> Net-(S7-Pad1)
- S7 pad 7: Net-(S7-Pad3) -> Net-(S7-Pad1)
- S8 pad 5: Net-(S8-Pad5) -> Net-(S8-Pad1)
- S8 pad 7: Net-(S8-Pad3) -> Net-(S8-Pad1)
- U1 pad 1: Net-(S5-Pad5) -> Net-(S5-Pad1)
- U1 pad 10: Net-(S12-Pad1) -> Net-(S12-Pad3)
- U1 pad 11: Net-(S12-Pad5) -> Net-(S12-Pad7)
- U1 pad 12: Net-(S13-Pad1) -> Net-(S13-Pad3)
- U1 pad 13: Net-(S13-Pad5) -> Net-(S13-Pad7)
- U1 pad 2: Net-(S5-Pad1) -> Net-(S5-Pad3)
- U1 pad 3: Net-(S6-Pad5) -> Net-(S6-Pad1)
- U1 pad 4: Net-(S6-Pad1) -> Net-(S6-Pad3)
- U1 pad 5: Net-(S7-Pad5) -> Net-(S7-Pad1)
- U1 pad 6: Net-(S7-Pad1) -> Net-(S7-Pad3)
- U1 pad 8: Net-(S8-Pad1) -> Net-(S8-Pad3)
- U1 pad 9: Net-(S8-Pad5) -> Net-(S8-Pad1)
- U10 pad 1: RES -> /RES
- U11 pad 1: D7 -> /D7
- U11 pad 10: (no net) -> unconnected-(U11-Pad10)
- U11 pad 11: (no net) -> unconnected-(U11-Pad11)
- U11 pad 12: (no net) -> unconnected-(U11-Pad12)
- U11 pad 13: (no net) -> unconnected-(U11-Pad13)
- U11 pad 8: (no net) -> unconnected-(U11-Pad8)
- U11 pad 9: (no net) -> unconnected-(U11-Pad9)
- U12 pad 1: D7 -> /D7
- U12 pad 8: D7 -> /D7
- U13 pad 2: RES -> /RES
- U3 pad 1: Net-(S14-Pad5) -> Net-(S14-Pad7)
- U3 pad 11: D7 -> /D7
- U3 pad 2: Net-(S14-Pad1) -> Net-(S14-Pad3)
- U3 pad 3: RES -> /RES
- U3 pad 5: (no net) -> unconnected-(U3-Pad5)
- U3 pad 6: (no net) -> unconnected-(U3-Pad6)
- U3 pad 8: Net-(S18-Pad1) -> Net-(S18-Pad3)
- U5 pad 2: RES -> /Input-Output/RST
- U6 pad 12: D7 -> /D7
- U6 pad 14: A1 -> /A1
- U6 pad 15: A2 -> /A2
- U6 pad 25: RES -> /RES
- U7 pad 1: A1 -> /A2
- U7 pad 2: A2 -> /A1
- U8 pad 19: D7 -> /CPU/D7
- U8 pad 8: A2 -> /A1
- U8 pad 9: A1 -> /A2
Other:
- board text removed: "(TMR0-OUT)"
- board text removed: "(TMR0-TRIG)"
- board text removed: "0"
- board text removed: "6"
- board text removed: "7"
- board text removed: "ADDR"
- board text removed: "CLK"
- board text removed: "DATA"
- board text removed: "HI"
- board text removed: "IN0"
- board text removed: "IN1"
- board text removed: "IN2"
- board text removed: "IN3"
- board text removed: "IN4"
- board text removed: "IN5"
- board text removed: "IN6"
- board text removed: "IN7"
- board text removed: "LO"
- board text removed: "OUT"
- board text removed: "PLC14500 Nano"
- board text removed: "R"
- board text removed: "RST"
- board text removed: "RUN"
- board text removed: "SPR"
- board text removed: "ST"
- board text removed: "STEP"
- board text removed: "TMR0"

Commit message: REV.D first proto
Parts:
- C4, C7: footprint Capacitor_THT:CP_Radial_D8.0mm_P5.00mm -> Capacitor_THT:CP_Radial_D5.0mm_P2.50mm
- moved R1 89.8 mm to (182.0, 133.4)
- moved D1 89.8 mm to (174.7, 122.1)
- moved R5 89.8 mm to (169.6, 133.4)
- moved S1 89.8 mm to (172.2, 128.3)
- moved S5 89.8 mm to (172.0, 140.9)
- moved R11 88.2 mm to (92.8, 133.4)
- moved S11 88.2 mm to (82.6, 128.3)
- moved S14 88.2 mm to (82.4, 140.9)
- moved D7 88.2 mm to (85.2, 122.1)
- moved R14 88.2 mm to (80.3, 133.4)
- moved D2 60.2 mm to (159.8, 122.1)
- moved R6 60.2 mm to (154.7, 133.4)
- moved R2 60.2 mm to (167.2, 133.4)
- moved S2 60.2 mm to (157.3, 128.3)
- moved S6 60.2 mm to (157.1, 140.9)
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- renumbered RV1 to locked
Connections:
- S12 pad 8: (no net) -> GND
- S12 pad 9: (no net) -> GND
- S13 pad 8: (no net) -> GND
- S13 pad 9: (no net) -> GND
- S14 pad 8: (no net) -> GND
- S14 pad 9: (no net) -> GND
- S16 pad 8: (no net) -> GND
- S16 pad 9: (no net) -> GND
- S18 pad 8: (no net) -> GND
- S18 pad 9: (no net) -> GND
- S5 pad 8: (no net) -> GND
- S5 pad 9: (no net) -> GND
- S6 pad 8: (no net) -> GND
- S6 pad 9: (no net) -> GND
- S7 pad 8: (no net) -> GND
- S7 pad 9: (no net) -> GND
- S8 pad 8: (no net) -> GND
- S8 pad 9: (no net) -> GND
Routing:
- net +5V: track 0.00 -> 651.3 mm
- net /TMR0-TRG: track 0.00 -> 237.9 mm
- net /A4: track 0.00 -> 214.2 mm, vias 0 -> 1
- net /D4: track 0.00 -> 205.1 mm, vias 0 -> 3
- net /A6: track 0.00 -> 203.2 mm
- net /A5: track 0.00 -> 202.7 mm
- net /Input-Output/EXTIN6: track 0.00 -> 200.9 mm, vias 0 -> 1
- net /D5: track 0.00 -> 199.6 mm, vias 0 -> 2
- net /A3: track 0.00 -> 198.8 mm, vias 0 -> 1
- net /D6: track 0.00 -> 196.2 mm, vias 0 -> 2
- net /A7: track 0.00 -> 191.0 mm, vias 0 -> 1
- net /Input-Output/EXTIN5: track 0.00 -> 188.7 mm, vias 0 -> 1
- net /A2: track 0.00 -> 187.0 mm, vias 0 -> 1
- net /RES: track 0.00 -> 179.9 mm, vias 0 -> 1
- net /A1: track 0.00 -> 178.1 mm, vias 0 -> 1
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Other:
- board text added: "I/O Expansion"
- board text added: "PLC14500 Nano"
- board text added: "TMR0-OUT"
- board text added: "WARNING! Logical signals only. DO NOT connect loads!"
- board text removed: "REV.C"

Commit message: Fixes
Parts:
- added C15: 100nF, Capacitor_THT:C_Rect_L7.2mm_W2.5mm_P5.00mm_FKS2_FKP2_MKS2_MKP2, F.Cu at (120.7, 117.5)
- added R59: 820R, Resistor_THT:R_Axial_DIN0204_L3.6mm_D1.6mm_P7.62mm_Horizontal, F.Cu at (108.0, 117.5)
Connections:
- D22 pad A: /A2 -> /A1
- D24 pad A: /A1 -> /A2
- D37 pad A: /CPU/D7 -> /D7
- J1 pad 17: /Input-Output/RST -> /RES
- U11 pad 10: unconnected-(U11-Pad10) -> Net-(U11-Pad10)
- U11 pad 11: unconnected-(U11-Pad11) -> Net-(U11-Pad11)
- U11 pad 8: unconnected-(U11-Pad8) -> Net-(U11-Pad11)
- U11 pad 9: unconnected-(U11-Pad9) -> Net-(C15-Pad1)
- U12 pad 2: /W -> Net-(U11-Pad10)
- U12 pad 5: /W -> Net-(U11-Pad10)
- U5 pad 2: /Input-Output/RST -> /RES
- U7 pad 1: /A2 -> /A1
- U7 pad 2: /A1 -> /A2
- U8 pad 19: /CPU/D7 -> /D7
- U8 pad 8: /A1 -> /A2
- U8 pad 9: /A2 -> /A1
Routing:
- net /D7: track 100.1 -> 191.6 mm, vias 0 -> 5
- net /RES: track 179.9 -> 262.9 mm
- net /Input-Output/RST: track 83.0 -> 0.00 mm
- net /CPU/D7: track 67.4 -> 0.00 mm
- net Net-(C15-Pad1): track 0.00 -> 41.0 mm, vias 0 -> 5
- net /W: track 106.8 -> 135.1 mm, vias 3 -> 5
- net Net-(S8-Pad3): track 58.5 -> 60.2 mm

Commit message: route
Parts:
- moved locked 51.4 mm to (218.4, 111.1)
- moved D10 31.8 mm to (225.4, 95.2)
- moved D11 31.8 mm to (225.4, 89.5)
- moved D12 31.8 mm to (225.3, 83.8)
- moved D13 31.8 mm to (225.3, 78.1)
- moved D14 31.8 mm to (225.3, 72.4)
- moved D15 31.8 mm to (225.3, 66.7)
- moved D9 31.8 mm to (225.4, 101.0)
- moved locked 31.8 mm to (214.5, 101.0)
- moved locked 31.8 mm to (214.5, 95.2)
- moved locked 31.8 mm to (214.5, 89.5)
- moved locked 31.8 mm to (214.4, 83.8)
- moved locked 31.8 mm to (214.4, 78.1)
- moved locked 31.8 mm to (214.4, 72.3)
- moved locked 31.8 mm to (214.4, 66.6)
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- renumbered R17 to locked, R33 to locked, R60 to locked, J1 to locked, R18 to locked, R19 to locked, R20 to locked, R21 to locked, R23 to locked, R24 to locked, R25 to locked, R32 to locked
Routing:
- net /Input-Output/EXTIN2: track 163.3 -> 98.3 mm
- net Net-(U13-Q3): track 72.6 -> 124.4 mm, vias 2 -> 7
- net /Input-Output/EXTIN0: track 111.2 -> 66.3 mm
- net /Input-Output/EXTIN5: track 188.7 -> 145.1 mm, vias 1 -> 0
- net Net-(U4-TRI): track 169.7 -> 126.7 mm
- net /Input-Output/OUT0: track 47.3 -> 89.0 mm
- net /Input-Output/OUT6: track 109.2 -> 67.6 mm, vias 0 -> 1
- net /Input-Output/EXTIN4: track 169.6 -> 128.0 mm, vias 1 -> 0
- net /Input-Output/EXTIN1: track 121.6 -> 80.4 mm
- net /Input-Output/OUT1: track 47.6 -> 88.1 mm
- net /Input-Output/EXTIN3: track 153.2 -> 113.9 mm, vias 1 -> 0
- net Net-(S5-Pad3): track 112.9 -> 151.8 mm
- net /Input-Output/OUT2: track 58.3 -> 93.8 mm, vias 0 -> 1
- net /Input-Output/EXTIN6: track 200.9 -> 167.7 mm, vias 1 -> 0
- net Net-(U11-Pad10): track 0.00 -> 32.1 mm
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Other:
- board size 160.1 x 99.9 mm -> 160.1 x 101 mm
- board text removed: "I/O Expansion"
- board text removed: "WARNING! Logical signals only. DO NOT connect loads!"
