File: board/plc14500/plc14500.kicad_pcb (KiCad board)
At the start: 2 copper layers, 160.1 x 101 mm, 173 parts, among them U1 74HC14, U10 MC14500, U11 74HC14, U12 4011, U13 4099, U14 4051, U2 4051, U3 74HC14, U4 NE555, U5 4099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

Commit message: Added reset cap from program line
Parts:
- added C20: 1uF NP, Capacitor_THT:C_Radial_D6.3mm_H5.0mm_P2.50mm, F.Cu at (115.6, 52.7)
Routing:
- net /PRG: track 106.0 -> 130.9 mm, vias 0 -> 2
- net /RES: track 249.6 -> 268.2 mm
